File: ESP32_Sensor_Board/main.brd (EAGLE design)
At the start: 100 x 80 mm, 2 parts

Commit message: Update com o projeto atualizado no eagle
Routing:
- net GND: track 27.1 -> 1.80 mm
- net SDA: track 32.9 -> 40.3 mm
- net SCL: track 29.3 -> 28.4 mm
- added copper zone on layer 16, net GND
Changed lines of the file:
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@@
 <layer number="43" name="vRestrict" color="2" fill="10" visible="yes" active="yes"/>
 <layer number="44" name="Drills" color="7" fill="1" visible="no" active="yes"/>
-<layer number="45" name="Holes" color="7" fill="1" visible="no" active="yes"/>
+<layer number="45" name="Holes" color="7" fill="1" visible="yes" active="yes"/>
 <layer number="46" name="Milling" color="3" fill="1" visible="no" active="yes"/>
 <layer number="47" name="Measures" color="7" fill="1" visible="no" active="yes"/>
@@
 <wire x1="100" y1="80" x2="0" y2="80" width="0" layer="20"/>
 <wire x1="0" y1="80" x2="0" y2="0" width="0" layer="20"/>
+<hole x="1.27" y="1.27" drill="0.35"/>
+<hole x="99.06" y="1.27" drill="0.35"/>
+<hole x="99.06" y="78.74" drill="0.35"/>
+<hole x="1.27" y="78.74" drill="0.35"/>
 </plain>
 <attributes>
@@
 <contactref element="U$1" pad="VCC"/>
 <contactref element="U$2" pad="3.3V"/>
-<wire x1="57.15" y1="50.8" x2="57.15" y2="60.96" width="1.27" layer="16"/>
-<wire x1="57.15" y1="60.96" x2="59.69" y2="63.5" width="1.27" layer="16"/>
+<wire x1="57.15" y1="50.8" x2="57.15" y2="60.96" width="1.27" layer="1"/>
+<wire x1="57.15" y1="60.96" x2="59.69" y2="63.5" width="1.27" layer="1"/>
 </signal>
 <signal name="GND">
@@
 <contactref element="U$2" pad="GND2"/>
 <wire x1="80.01" y1="50.8" x2="78.74" y2="49.53" width="1.27" layer="16"/>
-<wire x1="78.74" y1="49.53" x2="71.12" y2="49.53" width="1.27" layer="16"/>
-<wire x1="71.12" y1="49.53" x2="62.23" y2="58.42" width="1.27" layer="16"/>
-<wire x1="62.23" y1="58.42" x2="62.23" y2="63.5" width="1.27" layer="16"/>
+<polygon width="1.27" layer="16">
+<vertex x="0" y="80.01"/>
+<vertex x="0" y="0"/>
+<vertex x="100.33" y="0"/>
+<vertex x="100.33" y="80.01"/>
+</polygon>
 </signal>
 <signal name="SCL">
 <contactref element="U$2" pad="GPIO23"/>
 <contactref element="U$1" pad="SCL"/>
-<wire x1="80.01" y1="48.26" x2="81.28" y2="49.53" width="1.27" layer="16"/>
-<wire x1="81.28" y1="49.53" x2="82.55" y2="49.53" width="1.27" layer="16"/>
-<wire x1="82.55" y1="49.53" x2="82.55" y2="53.34" width="1.27" layer="16"/>
-<wire x1="82.55" y1="53.34" x2="81.28" y2="54.61" width="1.27" layer="16"/>
-<wire x1="81.28" y1="54.61" x2="71.12" y2="54.61" width="1.27" layer="16"/>
-<wire x1="71.12" y1="54.61" x2="67.31" y2="58.42" width="1.27" layer="16"/>
-<wire x1="67.31" y1="58.42" x2="67.31" y2="63.5" width="1.27" layer="16"/>
+<wire x1="67.31" y1="63.5" x2="75.0824" y2="55.7276" width="1.27" layer="1"/>
+<wire x1="75.0824" y1="55.7276" x2="82.55" y2="55.7276" width="1.27" layer="1"/>
+<wire x1="82.55" y1="55.7276" x2="82.55" y2="48.4124" width="1.27" layer="1"/>
+<wire x1="82.55" y1="48.4124" x2="80.69081875" y2="48.4124" width="1.27" layer="1"/>
+<wire x1="80.69081875" y1="48.4124" x2="80.53841875" y2="48.26" width="1.27" layer="1"/>
+<wire x1="80.53841875" y1="48.26" x2="80.01" y2="48.26" width="1.27" layer="1"/>
 </signal>
 <signal name="SDA">
@@
 <wire x1="80.01" y1="45.72" x2="81.28" y2="46.99" width="1.27" layer="16"/>
 <wire x1="81.28" y1="46.99" x2="85.09" y2="46.99" width="1.27" layer="16"/>
-<wire x1="85.09" y1="46.99" x2="85.09" y2="55.88" width="1.27" layer="16"/>
 <wire x1="85.09" y1="55.88" x2="83.82" y2="57.15" width="1.27" layer="16"/>
-<wire x1="83.82" y1="57.15" x2="76.2" y2="57.15" width="1.27" layer="16"/>
-<wire x1="76.2" y1="57.15" x2="69.85" y2="63.5" width="1.27" layer="16"/>
+<wire x1="69.85" y1="63.5" x2="76.2" y2="57.15" width="1.27" layer="1"/>
+<wire x1="76.2" y1="57.15" x2="83.82" y2="57.15" width="1.27" layer="1"/>
+<wire x1="83.82" y1="57.15" x2="85.09" y2="55.88" width="1.27" layer="1"/>
+<wire x1="85.09" y1="55.88" x2="85.09" y2="46.99" width="1.27" layer="1"/>
+<wire x1="85.09" y1="46.99" x2="81.28" y2="46.99" width="1.27" layer="1"/>
+<wire x1="81.28" y1="46.99" x2="80.01" y2="45.72" width="1.27" layer="1"/>
+<wire x1="85.09" y1="46.99" x2="85.09" y2="55.88" width="0" layer="19" extent="16-16"/>
 </signal>
 </signals>
